Commit message: Update _D435.urdf.xacro

File: megatrond_descripton/urdf/_D435.urdf.xacro (robot description, xacro)
@@ -8,5 +8,5 @@
 <robot name="sensor_d435" xmlns:xacro="http://ros.org/wiki/xacro">
   <!--File includes-->
-  <xacro:include filename="$(find megatrond_description)/urdf/_D435.gazebo.xacro">
+  <xacro:include filename="$(find megatrond_description)/urdf/_D435.gazebo.xacro"/>
   <xacro:macro name="sensor_d435" params="name:=camera topics_ns:=camera parent *origin">
     <xacro:property name="M_PI" value="3.1415926535897931" />
@@ -47,6 +47,6 @@
       <origin xyz="${d435_cam_mount_from_center_offset} ${-d435_cam_depth_py} 0" rpy="${M_PI/2} 0 ${M_PI/2}"/>
         <geometry>
-          <!-- <box size="${d435_cam_width} ${d435_cam_height} ${d435_cam_depth}"/> -->
-          <mesh filename="package://realsense2_description/meshes/d435.dae" />
+          <box size="${d435_cam_width} ${d435_cam_height} ${d435_cam_depth}"/>
+          <!--<mesh filename="package://megatrond_description/meshes/d435.dae" /> -->
           <!--<mesh filename="package://realsense2_description/meshes/d435/d435.dae" />-->
         </geometry>
